Commit message: agent_sim change1

File: clcbs_gazebo/models/agent/urdf/agent_sim.xacro (robot description, xacro)
@@ -82,5 +82,5 @@
         <parent link="robot_base" />
         <child link="course_agv__imu" />
-        <origin rpy="0  0  0" xyz="0.0 0.0 ${height/2+chassis_height}" />
+        <origin rpy="0  0  0" xyz="0.0 0.0 ${height/2 + chassis_height}" />
         <axis xyz="0  0  0" />
         <limit effort="0" lower="0" upper="0" velocity="0" />
@@ -119,5 +119,5 @@
         </inertial>
         <collision name="course_agv__collision">
-            <origin rpy="0 0 0" xyz="${-(length/2-base_to_back)} 0.0 ${height/2.0+chassis_height}" />
+            <origin rpy="0 0 0" xyz="${-length/2 - base_to_back} 0.0 ${height / 2.0 + chassis_height}" />
             <geometry>
                 <box size="${length} ${width} ${height}" />
@@ -125,5 +125,5 @@
         </collision>
         <visual>
-            <origin rpy="0 0 0" xyz="${-(length/2-base_to_back)} 0.0 ${height/2.0+chassis_height}" />
+            <origin rpy="0 0 0" xyz="${-length / 2 + base_to_back} 0.0 ${height / 2.0 + chassis_height}" />
             <geometry>
                 <box size="${length} ${width} ${height}" />
@@ -132,11 +132,11 @@
         </visual>
         <collision name="course_agv__left_caster_collision">
-            <origin rpy="0 0 0" xyz="${-base_to_caster} ${width/2-caster_radius} ${caster_radius}" />
-            <geometry>
-                <sphere radius="${caster_radius}" />
-            </geometry>
-        </collision>
-        <visual>
-            <origin rpy="0 0 0" xyz="${-base_to_caster} ${width/2-caster_radius} ${caster_radius}" />
+            <origin rpy="0 0 0" xyz="${-base_to_caster} ${width / 2 - caster_radius} ${caster_radius}" />
+            <geometry>
+                <sphere radius="${caster_radius}" />
+            </geometry>
+        </collision>
+        <visual>
+            <origin rpy="0 0 0" xyz="${-base_to_caster} ${width / 2 - caster_radius} ${caster_radius}" />
             <geometry>
                 <sphere radius="${caster_radius}" />
@@ -145,11 +145,11 @@
         </visual>
         <collision name="course_agv__right_caster_collision">
-            <origin rpy="0 0 0" xyz="${-base_to_caster} ${-(width/2-caster_radius)} ${caster_radius}" />
-            <geometry>
-                <sphere radius="${caster_radius}" />
-            </geometry>
-        </collision>
-        <visual>
-            <origin rpy="0 0 0" xyz="${-base_to_caster} ${-(width/2-caster_radius)} ${caster_radius}" />
+            <origin rpy="0 0 0" xyz="${-base_to_caster} ${-width / 2 + caster_radius} ${caster_radius}" />
+            <geometry>
+                <sphere radius="${caster_radius}" />
+            </geometry>
+        </collision>
+        <visual>
+            <origin rpy="0 0 0" xyz="${-base_to_caster} ${-width / 2 + caster_radius} ${caster_radius}" />
             <geometry>
                 <sphere radius="${caster_radius}" />

Commit message: agent_sim change2

File: clcbs_gazebo/models/agent/urdf/agent_sim.xacro (robot description, xacro)
@@ -36,5 +36,5 @@
             <inertia ixx="0" ixy="0" ixz="0" iyy="0" iyz="0" izz="0" />
         </inertial>
-        <collision name="course_agv__collision">
+        <collision>
             <origin rpy="0 0 0" xyz="0.0 0.0 0.0" />
             <geometry>
@@ -64,5 +64,5 @@
             <inertia ixx="0" ixy="0" ixz="0" iyy="0" iyz="0" izz="0" />
         </inertial>
-        <collision name="course_agv__collision">
+        <collision>
             <origin rpy="0 0 0" xyz="0.0 0.0 0.0" />
             <geometry>
@@ -118,5 +118,5 @@
             <inertia ixx="${mass / 12.0 * (width*width+height*height)}" ixy="0" ixz="0" iyy="${mass / 12.0 * (length*length + height*height)}" iyz="0" izz="${mass / 12.0 * (width*width + length*length)}" />
         </inertial>
-        <collision name="course_agv__collision">
+        <collision>
             <origin rpy="0 0 0" xyz="${-length/2 - base_to_back} 0.0 ${height / 2.0 + chassis_height}" />
             <geometry>
@@ -131,5 +131,5 @@
             <material name="yellow" />
         </visual>
-        <collision name="course_agv__left_caster_collision">
+        <collision>
             <origin rpy="0 0 0" xyz="${-base_to_caster} ${width / 2 - caster_radius} ${caster_radius}" />
             <geometry>
@@ -144,5 +144,5 @@
             <material name="yellow" />
         </visual>
-        <collision name="course_agv__right_caster_collision">
+        <collision>
             <origin rpy="0 0 0" xyz="${-base_to_caster} ${-width / 2 + caster_radius} ${caster_radius}" />
             <geometry>

Commit message: agent_sim.xacro change2 why changing link names cause the invalidity of material???

File: clcbs_gazebo/models/agent/urdf/agent_sim.xacro (robot description, xacro)
@@ -23,5 +23,5 @@
     <link name="robot_base" />
     <!-- left wheel -->
-    <joint name="course_agv__left_wheel_joint" type="continuous">
+    <joint name="agent_leftwheel_joint" type="continuous">
         <parent link="robot_base" />
         <child link="course_agv__left_wheel" />
@@ -51,5 +51,5 @@
     </link>
     <!-- right wheel -->
-    <joint name="course_agv__right_wheel_joint" type="continuous">
+    <joint name="agent_rightwheel_joint" type="continuous">
         <parent link="robot_base" />
         <child link="course_agv__right_wheel" />
@@ -79,5 +79,5 @@
     </link>
     <!-- imu -->
-    <joint name="course_agv__imu_joint" type="fixed">
+    <joint name="agent_imu_joint" type="fixed">
         <parent link="robot_base" />
         <child link="course_agv__imu" />
@@ -107,5 +107,5 @@
     </link>
     <!-- chassis -->
-    <joint name="course_agv__chassis_joint" type="fixed">
+    <joint name="agent_chassis_joint" type="fixed">
         <parent link="robot_base" />
         <child link="robot_chassis" />
@@ -186,5 +186,5 @@
     <transmission name="tran_left_wheel">
         <type>transmission_interface/SimpleTransmission</type>
-        <joint name="course_agv__left_wheel_joint">
+        <joint name="agent_leftwheel_joint">
             <hardwareInterface>hardware_interface/VelocityJointInterface</hardwareInterface>
         </joint>
@@ -196,5 +196,5 @@
     <transmission name="tran_right_wheel">
         <type>transmission_interface/SimpleTransmission</type>
-        <joint name="course_agv__right_wheel_joint">
+        <joint name="agent_rightwheel_joint">
             <hardwareInterface>hardware_interface/VelocityJointInterface</hardwareInterface>
         </joint>

Commit message: link name change complete

File: clcbs_gazebo/models/agent/urdf/agent_sim.xacro (robot description, xacro)
@@ -25,10 +25,10 @@
     <joint name="agent_leftwheel_joint" type="continuous">
         <parent link="robot_base" />
-        <child link="course_agv__left_wheel" />
+        <child link="agent_leftwheel_link" />
         <origin rpy="0 ${PI/2.0} ${PI/2.0}" xyz="0.0 ${(width / 2.0 + wheel_thickness / 2.0)} ${wheel_radius}" />
         <axis xyz="9.00000000e-05   9.00000000e-05   1.00000000e+00" />
         <limit effort="100" lower="0" upper="0" velocity="10" />
     </joint>
-    <link name="course_agv__left_wheel">
+    <link name="agent_leftwheel_link">
         <inertial>
             <mass value="${wheel_mass}" />
@@ -53,10 +53,10 @@
     <joint name="agent_rightwheel_joint" type="continuous">
         <parent link="robot_base" />
-        <child link="course_agv__right_wheel" />
+        <child link="agent_rightwheel_link" />
         <origin rpy="0 ${PI/2.0} ${PI/2.0}" xyz="0.0 ${-(width / 2.0 + wheel_thickness / 2.0)}  ${wheel_radius}" />
         <axis xyz="9.00000000e-05   9.00000000e-05   1.00000000e+00" />
         <limit effort="100" lower="0" upper="0" velocity="10" />
     </joint>
-    <link name="course_agv__right_wheel">
+    <link name="agent_rightwheel_link">
         <inertial>
             <mass value="${wheel_mass}" />
@@ -81,10 +81,10 @@
     <joint name="agent_imu_joint" type="fixed">
         <parent link="robot_base" />
-        <child link="course_agv__imu" />
+        <child link="agent_imu_link" />
         <origin rpy="0  0  0" xyz="0.0 0.0 ${height/2 + chassis_height}" />
         <axis xyz="0  0  0" />
         <limit effort="0" lower="0" upper="0" velocity="0" />
     </joint>
-    <link name="course_agv__imu">
+    <link name="agent_imu_link">
         <collision>
             <origin xyz="0 0 0" rpy="0 0 0" />
@@ -116,5 +116,6 @@
             <mass value="${mass}" />
             <origin rpy="0 0 0" xyz="0 0 0" />
-            <inertia ixx="${mass / 12.0 * (width*width+height*height)}" ixy="0" ixz="0" iyy="${mass / 12.0 * (length*length + height*height)}" iyz="0" izz="${mass / 12.0 * (width*width + length*length)}" />
+            <inertia ixx="${mass / 12.0 * (width*width+height*height)}" ixy="0" ixz="0"
+                iyy="${mass / 12.0 * (length*length + height*height)}" iyz="0" izz="${mass / 12.0 * (width*width + length*length)}" />
         </inertial>
         <collision>

Commit message: The car is already controllable!!!

File: clcbs_gazebo/models/agent/urdf/agent_sim.xacro (robot description, xacro)
@@ -78,32 +78,4 @@
         </visual>
     </link>
-    <!-- imu -->
-    <joint name="agent_imu_joint" type="fixed">
-        <parent link="robot_base" />
-        <child link="agent_imu_link" />
-        <origin rpy="0  0  0" xyz="0.0 0.0 ${height/2 + chassis_height}" />
-        <axis xyz="0  0  0" />
-        <limit effort="0" lower="0" upper="0" velocity="0" />
-    </joint>
-    <link name="agent_imu_link">
-        <collision>
-            <origin xyz="0 0 0" rpy="0 0 0" />
-            <geometry>
-                <box size="0.02 0.02 0.01" />
-            </geometry>
-        </collision>
-        <visual>
-            <origin xyz="0 0 0" rpy="0 0 0" />
-            <geometry>
-                <box size="0.02 0.02 0.01" />
-            </geometry>
-            <material name="red" />
-        </visual>
-        <inertial>
-            <mass value="0.001" />
-            <origin xyz="0 0 0" rpy="0 0 0" />
-            <inertia ixx="0.00000015" ixy="0" ixz="0" iyy="0.00000015" iyz="0" izz="0.00000015" />
-        </inertial>
-    </link>
     <!-- chassis -->
     <joint name="agent_chassis_joint" type="fixed">
@@ -159,30 +131,4 @@
         </visual>
     </link>
-    <!-- hokuyo laser -->
-    <!-- <link name="course_agv__hokuyo__link">
-        <inertial>
-            <mass value="1e-5"/>
-            <origin rpy="0 0 0" xyz="0 0 0"/>
-            <inertia ixx="0" ixy="0" ixz="0" iyy="0" iyz="0" izz="0"/>
-        </inertial>
-        <collision name="course_agv__hokuyo__collision-base">
-            <origin rpy="0 0 0" xyz="0 0 -0.035"/>
-            <geometry>
-                <box size="0.05 0.05 0.041"/>
-            </geometry>
-        </collision>
-        <collision name="course_agv__hokuyo__collision-top">
-            <origin rpy="0 0 0" xyz="0 0 0"/>
-            <geometry>
-                <cylinder length="0.029" radius="0.021"/>
-            </geometry>
-        </collision>
-        <visual>
-            <origin rpy="0  0  0" xyz="0  0 -0.0205"/>
-            <geometry>
-                <mesh filename="package://course_agv_description/meshes/hokuyo.dae" scale="1.0 1.0 1.0"/>
-            </geometry>
-        </visual>
-    </link> -->
     <transmission name="tran_left_wheel">
         <type>transmission_interface/SimpleTransmission</type>

Commit message: turn around the model

File: clcbs_gazebo/models/agent/urdf/agent_sim.xacro (robot description, xacro)
@@ -92,5 +92,5 @@
         </inertial>
         <collision>
-            <origin rpy="0 0 0" xyz="${-length/2 - base_to_back} 0.0 ${height / 2.0 + chassis_height}" />
+            <origin rpy="0 0 0" xyz="${length/2 + base_to_back} 0.0 ${height / 2.0 + chassis_height}" />
             <geometry>
                 <box size="${length} ${width} ${height}" />
@@ -98,5 +98,5 @@
         </collision>
         <visual>
-            <origin rpy="0 0 0" xyz="${-length / 2 + base_to_back} 0.0 ${height / 2.0 + chassis_height}" />
+            <origin rpy="0 0 0" xyz="${length / 2 - base_to_back} 0.0 ${height / 2.0 + chassis_height}" />
             <geometry>
                 <box size="${length} ${width} ${height}" />
@@ -105,5 +105,5 @@
         </visual>
         <collision>
-            <origin rpy="0 0 0" xyz="${-base_to_caster} ${width / 2 - caster_radius} ${caster_radius}" />
+            <origin rpy="0 0 0" xyz="${base_to_caster} ${width / 2 - caster_radius} ${caster_radius}" />
             <geometry>
                 <sphere radius="${caster_radius}" />
@@ -111,5 +111,5 @@
         </collision>
         <visual>
-            <origin rpy="0 0 0" xyz="${-base_to_caster} ${width / 2 - caster_radius} ${caster_radius}" />
+            <origin rpy="0 0 0" xyz="${base_to_caster} ${width / 2 - caster_radius} ${caster_radius}" />
             <geometry>
                 <sphere radius="${caster_radius}" />
@@ -118,5 +118,5 @@
         </visual>
         <collision>
-            <origin rpy="0 0 0" xyz="${-base_to_caster} ${-width / 2 + caster_radius} ${caster_radius}" />
+            <origin rpy="0 0 0" xyz="${base_to_caster} ${-width / 2 + caster_radius} ${caster_radius}" />
             <geometry>
                 <sphere radius="${caster_radius}" />
@@ -124,5 +124,5 @@
         </collision>
         <visual>
-            <origin rpy="0 0 0" xyz="${-base_to_caster} ${-width / 2 + caster_radius} ${caster_radius}" />
+            <origin rpy="0 0 0" xyz="${base_to_caster} ${-width / 2 + caster_radius} ${caster_radius}" />
             <geometry>
                 <sphere radius="${caster_radius}" />

Commit message: add reset; add observer; note <inertia> changed; controller algorithm still don't work

File: clcbs_gazebo/models/agent/urdf/agent_sim.xacro (robot description, xacro)
@@ -3,5 +3,5 @@
 <robot name="course_agv" xmlns:xacro="http://www.ros.org/wiki/xacro">
     <xacro:property name="PI" value="3.1415926535897931" />
-    <xacro:property name="mass" value="30" />
+    <xacro:property name="mass" value="5" />
     <xacro:property name="length" value="3" />
     <xacro:property name="width" value="2" />
@@ -9,5 +9,5 @@
     <xacro:property name="chassis_height" value="0.2" />
     <xacro:property name="caster_radius" value="${chassis_height/2}" />
-    <xacro:property name="wheel_mass" value="0.1" />
+    <xacro:property name="wheel_mass" value="0.5" />
     <xacro:property name="wheel_radius" value="0.5" />
     <xacro:property name="wheel_thickness" value="${wheel_radius/3}" />
@@ -87,5 +87,5 @@
         <inertial>
             <mass value="${mass}" />
-            <origin rpy="0 0 0" xyz="0 0 0" />
+            <origin rpy="0 0 0" xyz="0.5 0.0 0.0" /> <!-- CHANGE HERE TO SEE INFLUENCE-->
             <inertia ixx="${mass / 12.0 * (width*width+height*height)}" ixy="0" ixz="0"
                 iyy="${mass / 12.0 * (length*length + height*height)}" iyz="0" izz="${mass / 12.0 * (width*width + length*length)}" />

Commit message: add mass to caster and fix xacro bugs

File: clcbs_gazebo/models/agent/urdf/agent_sim.xacro (robot description, xacro)
@@ -10,4 +10,5 @@
     <xacro:property name="caster_radius" value="${chassis_height/2}" />
     <xacro:property name="wheel_mass" value="0.5" />
+    <xacro:property name="caster_mass" value="${wheel_mass}" />
     <xacro:property name="wheel_radius" value="0.5" />
     <xacro:property name="wheel_thickness" value="${wheel_radius/3}" />
@@ -87,10 +88,10 @@
         <inertial>
             <mass value="${mass}" />
-            <origin rpy="0 0 0" xyz="0.5 0.0 0.0" /> <!-- CHANGE HERE TO SEE INFLUENCE-->
+            <origin rpy="0 0 0" xyz="${length / 2 - base_to_back} 0.0 ${height / 2.0 + chassis_height}" /> <!-- CHANGE HERE TO SEE INFLUENCE-->
             <inertia ixx="${mass / 12.0 * (width*width+height*height)}" ixy="0" ixz="0"
                 iyy="${mass / 12.0 * (length*length + height*height)}" iyz="0" izz="${mass / 12.0 * (width*width + length*length)}" />
         </inertial>
         <collision>
-            <origin rpy="0 0 0" xyz="${length/2 + base_to_back} 0.0 ${height / 2.0 + chassis_height}" />
+            <origin rpy="0 0 0" xyz="${length / 2 - base_to_back} 0.0 ${height / 2.0 + chassis_height}" />
             <geometry>
                 <box size="${length} ${width} ${height}" />
@@ -104,4 +105,10 @@
             <material name="yellow" />
         </visual>
+        <inertial>
+            <mass value="${caster_mass}" />
+            <origin rpy="0 0 0" xyz="${base_to_caster} ${width / 2 - caster_radius} ${caster_radius}" />
+            <inertia ixx="${2.0 / 5.0 * mass * caster_radius * caster_radius}" ixy="0" ixz="0"
+                iyy="${2.0 / 5.0 * mass * caster_radius * caster_radius}" iyz="0" izz="${2.0 / 5.0 * mass * caster_radius * caster_radius}" />
+        </inertial>
         <collision>
             <origin rpy="0 0 0" xyz="${base_to_caster} ${width / 2 - caster_radius} ${caster_radius}" />
@@ -117,4 +124,10 @@
             <material name="yellow" />
         </visual>
+        <inertial>
+            <mass value="${caster_mass}" />
+            <origin rpy="0 0 0" xyz="${base_to_caster} ${-width / 2 - caster_radius} ${caster_radius}" />
+            <inertia ixx="${2.0 / 5.0 * mass * caster_radius * caster_radius}" ixy="0" ixz="0"
+                iyy="${2.0 / 5.0 * mass * caster_radius * caster_radius}" iyz="0" izz="${2.0 / 5.0 * mass * caster_radius * caster_radius}" />
+        </inertial>
         <collision>
             <origin rpy="0 0 0" xyz="${base_to_caster} ${-width / 2 + caster_radius} ${caster_radius}" />

Commit message: mid2: fix bugs; turn reversely;

File: clcbs_gazebo/models/agent/urdf/agent_sim.xacro (robot description, xacro)
@@ -3,5 +3,5 @@
 <robot name="course_agv" xmlns:xacro="http://www.ros.org/wiki/xacro">
     <xacro:property name="PI" value="3.1415926535897931" />
-    <xacro:property name="mass" value="5" />
+    <xacro:property name="mass" value="50" />
     <xacro:property name="length" value="3" />
     <xacro:property name="width" value="2" />

Commit message: stable 6.0 1. Rewrite CarModel to Linear-Turning 2. Modify Model to a Songling-like Car 3. Debug

File: clcbs_gazebo/models/agent/urdf/agent_sim.xacro (robot description, xacro)
@@ -4,15 +4,15 @@
     <xacro:property name="PI" value="3.1415926535897931" />
     <xacro:property name="mass" value="50" />
-    <xacro:property name="length" value="3" />
-    <xacro:property name="width" value="2" />
-    <xacro:property name="height" value="1" />
-    <xacro:property name="chassis_height" value="0.2" />
+    <xacro:property name="length" value="0.978" />
+    <xacro:property name="width" value="0.376" />
+    <xacro:property name="height" value="0.33" />
+    <xacro:property name="chassis_height" value="0.103" />
     <xacro:property name="caster_radius" value="${chassis_height/2}" />
     <xacro:property name="wheel_mass" value="0.5" />
     <xacro:property name="caster_mass" value="${wheel_mass}" />
-    <xacro:property name="wheel_radius" value="0.5" />
-    <xacro:property name="wheel_thickness" value="${wheel_radius/3}" />
-    <xacro:property name="base_to_back" value="1.0" />
-    <xacro:property name="base_to_caster" value="1.5" />
+    <xacro:property name="wheel_radius" value="0.164" />
+    <xacro:property name="wheel_thickness" value="0.1725" />
+    <xacro:property name="base_to_back" value="0.1725" />
+    <xacro:property name="base_to_caster" value="0.6" />
     <xacro:property name="center_span" value="0.0" />
     <xacro:property name="urdf_src" value="$(find clcbs_gazebo)/models/agent/urdf/" />
